Commit message: third commit

File: agv_description/urdf/agv.xacro (robot description, xacro)
@@ -278,3 +278,37 @@
     </sensor>
   </gazebo>
+ <link name="imu_link"/>
+<joint name="imu_joint" type="fixed">
+<parent link="base_link"/>
+<child link="imu_link"/>
+<origin xyz="0 0 0.1" rpy="0 0 0"/>
+</joint>
+<gazebo>
+<plugin name="imu_plugin" filename="libgazebo_ros_imu.so">
+<alwaysOn>true</alwaysOn>
+<bodyName>imu_link</bodyName>
+<frameName>imu_link</frameName>
+<topicName>imu</topicName>
+<serviceName>imu_service</serviceName>
+<gaussianNoise>0.0</gaussianNoise>
+<updateRate>200</updateRate>
+<imu>
+<noise>
+<type>gaussian</type>
+<rate>
+<mean>0.0</mean>
+<stddev>2e-4</stddev>
+<bias_mean>0.0000075</bias_mean>
+<bias_stddev>0.0000008</bias_stddev>
+</rate>
+<accel>
+<mean>0.0</mean>
+<stddev>1.7e-2</stddev>
+<bias_mean>0.1</bias_mean>
+<bias_stddev>0.001</bias_stddev>
+</accel>
+</noise>
+</imu>
+</plugin>
+</gazebo>
 </robot>

Commit message: 4 commit

File: agv_description/urdf/agv.xacro (robot description, xacro)
@@ -217,12 +217,12 @@
     </plugin>
   </gazebo>
-<joint name="hokuyo_joint" type="fixed">
+<joint name="scan_joint" type="fixed">
     <axis xyz="0 1 0" />
     <origin xyz="0 0 0.15" rpy="0 0 0"/>
     <parent link="base_link"/>
-    <child link="hokuyo_link"/>
+    <child link="base_scan"/>
   </joint>
   <!-- Hokuyo Laser -->
-  <link name="hokuyo_link">
+  <link name="base_scan">
     <collision>
       <origin xyz="0 0 0" rpy="${M_PI/2} 0 0"/>
@@ -243,5 +243,5 @@
     </inertial>
   </link>
-    <gazebo reference="hokuyo_link">
+    <gazebo reference="base_scan">
     <sensor type="gpu_ray" name="head_hokuyo_sensor">
       <pose>0 0 0 0 0 0</pose>
@@ -274,5 +274,5 @@
       <plugin name="gazebo_ros_head_hokuyo_controller" filename="libgazebo_ros_gpu_laser.so">
         <topicName>/scan</topicName>
-        <frameName>hokuyo_link</frameName>
+        <frameName>base_scan</frameName>
       </plugin>
     </sensor>
